File: pcb/pico v2.brd (EAGLE design)
At the start: 100 x 80 mm, 31 parts, among them IC3 74LS47N, IC4 74LS47N

Commit message: finetuning
Parts:
- added JP1: (no value), pinhead:1X05
Connections:
- new net N$28: JP1.1, U$1.29
- new net N$29: JP1.2, U$1.30
- new net N$35: JP1.3, U$1.31
- new net N$44: JP1.4, U$1.32
- new net N$48: JP1.5, U$1.33
- net VCC: no longer DIS1.5
Routing:
- net VCC: track 428.4 -> 346.4 mm
- net GND: track 384.5 -> 338.9 mm
- net N$44: track 0.00 -> 12.7 mm
- net N$48: track 0.00 -> 12.0 mm
- net N$35: track 0.00 -> 12.0 mm
- net N$29: track 0.00 -> 12.0 mm
- net N$28: track 0.00 -> 12.0 mm
- net N$43: track 19.1 -> 14.8 mm
- net N$8: track 47.7 -> 45.7 mm
Other:
- board text added: "DATA"
- board text added: "DIR"
- board text added: "EN"
- board text added: "GND"
- board text added: "VCC"
- board text added: "vcc"
