File: pcb/pico v2.sch (EAGLE design)
At the start: 31 parts, among them IC3 74LS47N, IC4 74LS47N

Commit message: finetuning
Parts:
- added JP1: (no value), pinhead:PINHD-1X5
Connections:
- new net N$28: JP1.1, U$1.29
- new net N$29: JP1.2, U$1.30
- new net N$35: JP1.3, U$1.31
- new net N$44: JP1.4, U$1.32
- new net N$48: JP1.5, U$1.33
- net VCC: no longer DIS1.DP
Other:
- moved on the sheet: DHT-11, LCD1, LED1, LED2, LED3, R1, R2, R3, R4

Commit message: .
Connections:
- net GND: now also U$1.8
Other:
- moved on the sheet: LED2, R2, R3, R4
