File: pcb/copie/pico v2 - Copy.brd (EAGLE design)
At the start: 100 x 80 mm, 32 parts, among them IC3 74LS47N, IC4 74LS47N

Commit message: .
Connections:
- net GND: no longer U$1.8
Routing:
- net GND: track 380.5 -> 338.9 mm
- net VCC: track 313.3 -> 346.4 mm
- net N$44: track 12.0 -> 12.7 mm
